File: Lab7/PCB_Schematic/Lab7/Lab7.kicad_sch (KiCad schematic)
At the start: 8 parts, among them J1 Conn_01x05_Pin, U1 TLC277

Commit message: Got signoffs
Parts:
- C1: value 0.68u -> 1.38u
- R3: value 480k -> 600k
Changed lines of the file:
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@@
 			)
 		)
-		(property "Value" "480k"
+		(property "Value" "600k"
 			(at 194.31 102.108 90)
 			(effects
@@
 			)
 		)
-		(property "Value" "0.68u"
+		(property "Value" "1.38u"
 			(at 168.656 93.726 0)
 			(effects
